File: docs/hardware/kicad/Esp32 relay.kicad_sch (KiCad schematic)
At the start: 83 parts, among them J1 Conn_01x05_Pin, J10 Screw_Terminal_01x04, J11 Screw_Terminal_01x05, J12 Screw_Terminal_01x04, J13 Screw_Terminal_01x05, J14 GPIO, J15 SPI, J2 Conn_01x05_Pin, J3 Screw_Terminal_01x02, J4 USB_C_Receptacle_USB2.0_16P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

Commit message: Updates PCB design to 1.2a
Parts:
- removed Flow1, Flow2, Pressure1, Pressure2: Conn_01x03_Pin, Connector_PinSocket_2.54mm:PinSocket_1x03_P2.54mm_Vertical, symbol Connector:Conn_01x03_Pin
- removed J1, J2: Conn_01x05_Pin, Connector_PinSocket_2.54mm:PinSocket_1x05_P2.54mm_Vertical, symbol Connector:Conn_01x05_Pin
- removed Led1, Led2: Conn_01x04_Socket, Connector_PinSocket_2.54mm:PinSocket_1x04_P2.54mm_Vertical, symbol Connector:Conn_01x04_Socket
- added D11, D12: D_TVS 3.3v, Diode_SMD:D_SOD-323_HandSoldering, symbol Device:D_TVS
- added F2, F3, F4, F5: 1.5A, Fuse:Fuse_1812_4532Metric_Pad1.30x3.40mm_HandSolder, symbol Device:Polyfuse_Small
- added Flow1, Flow2, Pressure1, Pressure2: Screw_Terminal_01x03, TerminalBlock_Phoenix:TerminalBlock_Phoenix_MKDS-1,5-3_1x03_P5.00mm_Horizontal, symbol Connector:Screw_Terminal_01x03
- F1: MANUFACTURER (none) -> Bel Fuse Inc.; Part# (none) -> 5923-0ZCG0150AF2CCT-ND; Price (none) -> 0.23300
- J10, J12: MANUFACTURER (none) -> Phoenix Contact; Part# (none) -> 1935187; Price (none) -> 1.03000
- J11, J13: MANUFACTURER (none) -> Phoenix Contact; Part# (none) -> 1935190; Price (none) -> 1.28000
- J3, J5, J6, J7, J8, J9: Price (none) -> .53000
- J4: MANUFACTURER (none) -> gtc
- K3, K4: Part# RF424F12 -> RT424F12-ND; Price None -> 10.00000
- R1, R11, R19: value 470R -> 1K; MANUFACTURER (none) -> Stackpole Electronics Inc; Part# (none) -> RMCF0805FT1K80CT-ND; Price (none) -> 0.01270
- R10, R13, R14, R15, R16, R17, R18, R20, R3, R4, R5, R6, R7, R8, R9: MANUFACTURER (none) -> Stackpole Electronics Inc
- R12, R2: value 470R -> 1.8K; MANUFACTURER (none) -> Stackpole Electronics Inc
- SW1, SW2, SW3, SW4: MANUFACTURER (none) -> E-Switch; Part# (none) -> 100DP3T1B3M2QEH-ND; Price (none) -> 4.52000
- SW5, SW6: MANUFACTURER (none) -> C&K; Part# (none) -> PTS636 SP50 SMTR LFS; Price (none) -> .23
- U1, U4: Price None -> .50800
- U2: Part# (none) -> 945-1036-ND; Price (none) -> 9.17000
- U3: Part# (none) -> 945-2201-ND; Price (none) -> 3.97000
- U6: MANUFACTURER (none) -> Espressif Systems; Part# (none) -> 5407-ESP32-S3-WROOM-1-N8R2CT-ND; Price (none) -> 5.88000
Connections:
- net 3v3: now also Flow1.1 (Pin_1), Flow2.1 (Pin_1)
- net 5V: now also Pressure1.1 (Pin_1), Pressure2.1 (Pin_1)
- net Earth: now also D11.1 (A1), D12.1 (A1), Flow1.3 (Pin_3), Flow2.3 (Pin_3), Pressure1.2 (Pin_2), Pressure2.2 (Pin_2)
- net GPIO1: now also D12.2 (A2)
- net GPIO2: now also D11.2 (A2)
- net GPIO38: now also Flow2.2 (Pin_2)
- net GPIO39: now also Flow1.2 (Pin_2)
- net at R10.2: now also Pressure1.3 (Pin_3)
- net at K3.11: now also F2.1; no longer J13.1 (Pin_1)
- net at K3.21: now also F3.1; no longer J13.2 (Pin_2)
- net at K4.11: now also F4.1; no longer J11.1 (Pin_1)
- net at J11.2 (Pin_2): now also F5.2; no longer K4.21
- net at R8.2: now also Pressure2.3 (Pin_3)
- new net: F2.2, J13.1 (Pin_1)
- new net: F3.2, J13.2 (Pin_2)
- new net: F4.2, J11.1 (Pin_1)
- new net: F5.1, K4.21
Other:
- moved on the sheet: J11, J12
